File: AstroEQ-Hardware/SMD/AstroEQ SMD MK2 (EQ5).sch (EAGLE design)
At the start: 41 parts, among them IC1 ATMEGA162-16AU, IC2 PIC18F14K50-I/SS, IC3 78L05, J1 POWER_JACKPANEL, M1 Motor Driver, M2 Motor Driver, SW1 SWITCH, X1 16MHz, X2 12MHz

Commit message: Added SMD design to fit inside EQ5 mount shell.
Parts:
- USB->: value Bulgin PX0458 -> Bulgin PX0447; MPN PX0458 -> PX0447; OC_FARNELL 1629391 -> 1229687
Other:
- moved on the sheet: C1, C10, C11, C12, C13, C14, C15, C2, C3, C4, C5, C6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
