File: AstroEQ-Hardware/SMD/AstroEQ SMD V4.7 (EQ5).brd (EAGLE design)
At the start: 85 x 49 mm, 53 parts, among them IC1 ATMEGA162-16AU, IC2 PIC18F14K50-I/SS, IC3 78L05, J1 POWER_JACKPANEL, M1 Motor Driver, M2 Motor Driver, Q1 NTR4501NT1G, X1 16MHz, X2 12MHz

Commit message: Update Hardware Designs
Minor corrections to part attributes and some components in the V4.7
design moved slightly to avoid collisions as found during the prototype
build.
Parts:
- D2: value PMEG2010EA -> RB511VM-30FHTE-17
- USB->: value Bulgin PX0443 -> MC34649
Changed lines of the file:
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@@
 <layer number="25" name="tNames" color="15" fill="1" visible="yes" active="yes"/>
 <layer number="26" name="bNames" color="7" fill="1" visible="yes" active="yes"/>
-<layer number="27" name="tValues" color="15" fill="1" visible="yes" active="yes"/>
-<layer number="28" name="bValues" color="7" fill="1" visible="yes" active="yes"/>
+<layer number="27" name="tValues" color="15" fill="1" visible="no" active="yes"/>
+<layer number="28" name="bValues" color="7" fill="1" visible="no" active="yes"/>
 <layer number="29" name="tStop" color="7" fill="3" visible="yes" active="yes"/>
 <layer number="30" name="bStop" color="7" fill="6" visible="yes" active="yes"/>
@@
 <layer number="49" name="Reference" color="7" fill="1" visible="no" active="yes"/>
 <layer number="50" name="dxf" color="7" fill="1" visible="no" active="no"/>
-<layer number="51" name="tDocu" color="7" fill="1" visible="yes" active="yes"/>
-<layer number="52" name="bDocu" color="7" fill="1" visible="yes" active="yes"/>
+<layer number="51" name="tDocu" color="7" fill="1" visible="no" active="yes"/>
+<layer number="52" name="bDocu" color="7" fill="1" visible="no" active="yes"/>
 <layer number="53" name="tGND_GNDA" color="7" fill="9" visible="no" active="no"/>
 <layer number="54" name="bGND_GNDA" color="1" fill="9" visible="no" active="no"/>
@@
 <attribute name="MPN" value="MCWR06X1002FTL" x="10.16" y="20.6375" size="1.778" layer="27" display="off"/>
 </element>
-<element name="USB-&gt;" library="adafruit" package="22-23-2051" value="Bulgin PX0443" x="4.1275" y="26.035" locked="yes" smashed="yes" rot="MR270">
+<element name="USB-&gt;" library="adafruit" package="22-23-2051" value="MC34649" x="4.1275" y="26.035" locked="yes" smashed="yes" rot="MR270">
 <attribute name="NAME" x="4.1275" y="33.655" size="1.27" layer="26" font="vector" ratio="15" rot="MR0" align="center"/>
-<attribute name="MF" value="BULGIN" x="4.1275" y="26.035" size="1.778" layer="28" rot="MR270" display="off"/>
-<attribute name="OC_FARNELL" value="1229685" x="4.1275" y="26.035" size="1.778" layer="28" rot="MR270" display="off"/>
-<attribute name="MPN" value="PX0443" x="4.1275" y="26.035" size="1.778" layer="28" rot="MR270" display="off"/>
+<attribute name="MF" value="MULTICOMP" x="4.1275" y="26.035" size="1.778" layer="28" rot="MR270" display="off"/>
+<attribute name="OC_FARNELL" value="1675777" x="4.1275" y="26.035" size="1.778" layer="28" rot="MR270" display="off"/>
+<attribute name="MPN" value="MC34649" x="4.1275" y="26.035" size="1.778" layer="28" rot="MR270" display="off"/>
 </element>
 <element name="C6" library="rcl" package="C0603" value="470n" x="8.255" y="29.5275" smashed="yes" rot="R270">
@@
 <attribute name="NAME" x="15.39875" y="23.84425" size="1.016" layer="25" font="vector" ratio="15" rot="R180" align="center"/>
 </element>
-<element name="D2" library="SparkFun" package="SOD-323" value="PMEG2010EA" x="3.175" y="33.655" smashed="yes">
-<attribute name="OC_FARNELL" value="8737908" x="3.175" y="33.655" size="1.778" layer="27" display="off"/>
-<attribute name="MF" value="NEXPERIA" x="3.175" y="33.655" size="1.778" layer="27" display="off"/>
-<attribute name="MPN" value="PMEG2010EA" x="3.175" y="33.655" size="1.778" layer="27" display="off"/>
+<element name="D2" library="SparkFun" package="SOD-323" value="RB511VM-30FHTE-17" x="3.175" y="33.655" smashed="yes">
+<attribute name="OC_FARNELL" value="2581544" x="3.175" y="33.655" size="1.778" layer="27" display="off"/>
+<attribute name="MF" value="ROHM" x="3.175" y="33.655" size="1.778" layer="27" display="off"/>
+<attribute name="MPN" value="RB511VM-30FHTE-17" x="3.175" y="33.655" size="1.778" layer="27" display="off"/>
 <attribute name="NAME" x="6.0325" y="33.655" size="1.016" layer="25" font="vector" ratio="15" align="center"/>
 </element>
