File: AstroEQ-Hardware/SMD/AstroEQ SMD V4.7 (EQ5).sch (EAGLE design)
At the start: 53 parts, among them IC1 ATMEGA162-16AU, IC2 PIC18F14K50-I/SS, IC3 78L05, J1 POWER_JACKPANEL, M1 Motor Driver, M2 Motor Driver, Q1 NTR4501NT1G, X1 16MHz, X2 12MHz

Commit message: Update AstroEQ PTH/SMD Schematics
1. Tidy up the schematics, add a frame, and improve labelling of nets
2. Add extra textual documentation to the PCB to label the various extra IO pins.
Parts:
- IC2: MPN PIC18F14K50-I/SS -> (none); PACKAGE SSOP20 -> (none)
- R15, R16: device SmartPrj:R-EU_R0603 -> rcl:R-EU_R0603
Other:
- moved on the sheet: C1, C10, C11, C12, C13, C14, C15, C16, C2, C3, C4, C5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
