File: AstroEQ-Hardware/SMD/AstroEQ SMD V4.8.brd (EAGLE design)
At the start: 100 x 66 mm, 55 parts, among them IC1 DIP40-SOCKET, IC2 DIP20-SOCKET, IC3 78L05, J2 DNI, J3 DNI, M1 Motor Driver, M2 Motor Driver, Q1 NTR4501NT1G, X1 16MHz, X2 12MHz

Commit message: Correct IO4 Pin on AstroEQ PCBs
Cannot use the Tx pin for this because the USB IC self-powers off this in standalone mode which prevents target speed selection.
Connections:
- new net IO4: IC1.21, R23.2
- net RX: no longer R23.2
Routing:
- net IO4: track 0.00 -> 32.8 mm
- net RX: track 29.8 -> 26.3 mm
- net GND: vias 170 -> 176
Other:
- board text added: "For DIY, use "AstroEQ PTH V4.8""
- board text removed: "For DIY, use "AstroEQ PTH V4.6""
Changed lines of the file:
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@@
 <wire x1="72.0725" y1="30.48" x2="72.0725" y2="29.21" width="0.254" layer="41"/>
 <text x="47.14875" y="30.48" size="1.27" layer="21" font="vector" ratio="15" align="center">1</text>
-<text x="0" y="69.85" size="1.778" layer="49" font="vector">For DIY, use "AstroEQ PTH V4.6"</text>
+<text x="0" y="69.85" size="1.778" layer="49" font="vector">For DIY, use "AstroEQ PTH V4.8"</text>
 <text x="47.46625" y="14.76375" size="1.2" layer="25" font="vector" ratio="15" align="center-left">GPIO:
 5: +5V
@@
 <via x="46.19625" y="25.4" extent="1-16" drill="0.5" shape="octagon"/>
 <via x="52.705" y="6.35" extent="1-16" drill="0.5" shape="octagon"/>
+<via x="28.575" y="43.18" extent="1-16" drill="0.5" shape="octagon"/>
+<via x="32.54375" y="46.0375" extent="1-16" drill="0.5" shape="octagon"/>
+<via x="28.575" y="48.26" extent="1-16" drill="0.5" shape="octagon"/>
+<via x="32.54375" y="50.4825" extent="1-16" drill="0.5" shape="octagon"/>
+<via x="46.99" y="29.845" extent="1-16" drill="0.5" shape="octagon"/>
+<via x="43.65625" y="27.94" extent="1-16" drill="0.5" shape="octagon"/>
 </signal>
 <signal name="V+">
@@
 <wire x1="30.48" y1="40.64" x2="41.91" y2="29.21" width="0.4064" layer="1"/>
 <wire x1="41.91" y1="29.21" x2="45.085" y2="29.21" width="0.4064" layer="1"/>
-<contactref element="R23" pad="2"/>
-<wire x1="45.085" y1="29.21" x2="47.0925" y2="31.2175" width="0.4064" layer="1"/>
-<wire x1="47.0925" y1="31.2175" x2="47.0925" y2="31.90875" width="0.4064" layer="1"/>
 </signal>
 <signal name="RX(USB)">
@@
 <wire x1="85.6775" y1="52.4375" x2="85.7275" y2="52.3875" width="0.4064" layer="1"/>
 </signal>
+<signal name="IO4">
+<contactref element="R23" pad="2"/>
+<contactref element="IC1" pad="21"/>
+<wire x1="47.0925" y1="31.90875" x2="45.66375" y2="30.48" width="0.4064" layer="1"/>
+<wire x1="45.66375" y1="30.48" x2="44.45" y2="30.48" width="0.4064" layer="1"/>
+<wire x1="44.45" y1="30.48" x2="43.97375" y2="30.00375" width="0.4064" layer="1"/>
+<wire x1="43.97375" y1="30.00375" x2="42.2275" y2="30.00375" width="0.4064" layer="1"/>
+<wire x1="42.2275" y1="30.00375" x2="31.4325" y2="40.79875" width="0.4064" layer="1"/>
+<wire x1="31.4325" y1="40.79875" x2="31.4325" y2="50.4825" width="0.4064" layer="1"/>
+<wire x1="31.4325" y1="50.4825" x2="29.845" y2="52.07" width="0.4064" layer="1"/>
+</signal>
 </signals>
