File: AstroEQ-Hardware/PTH/AstroEQ PTH MK3.sch (EAGLE design)
At the start: 46 parts, among them IC1 ATMEGA162-16PU, IC2 PIC18F14K50-I/P, IC3 78L05, J1 POWER_JACKPTH, M1 Motor Driver, M2 Motor Driver, X1 16MHz, X2 12MHz

Commit message: Update Hardware Files
Update the repository to contain the latest hardware designs for AstroEQ
V4.6, along with exported BOM.
Parts:
- added J2, J3: (no value), jumper:JUMPER
- added JP3, JP4: M01PTH, SparkFun:M01PTH
- added PWM: JACK, SparkFun:AUDIO-JACKPTH
- added Q1: BS270, SparkFun:MOSFET-NCHANNELPTH
- added R21: 1k, rcl:R-EU_0204/7
- added R22: 120, rcl:R-EU_0204/7
- added SJ1: (no value), jumper:JP2E
- added SJ2: (no value), jumper:JP2EL
- D1: MF CREE -> WOLFSPEED
- GPIO: MF (none) -> CYNERGY3; MPN (none) -> SSF211X050; OC_FARNELL (none) -> 4249100
- HAMMOND-1593N: value HAMMOND-1593N -> HAMMOND-1593N-4HOLE; device holes:HAMMOND-1593N -> holes:HAMMOND-1593N-4HOLE
- JP1, JP2, LOGO1: OC_FARNELL (none) -> unknown
- ST4: MF (none) -> MOLEX; MPN (none) -> 95501-2661; OC_FARNELL (none) -> 1536490
Connections:
- net DEC+ renamed DEC+/SI
- net DEC- renamed DEC-/CK
- net RA+ renamed RA+/SO
- net RA- renamed RA-/!SS
- new net MS13-1: M1.MS1(M0), SJ1.2
- new net MS13-2: M2.MS1(M0), SJ2.2
- new net N$2: PWM.RIGHT, Q1.D
- new net N$4: Q1.S, R22.2
- new net PWM: IC1.PB1/T1/OC2, JP3.1, JP4.1, Q1.G
- net !RST-1: now also M1.!RST; no longer M1.!RESET
- net !RST-2: now also M2.!RST; no longer M2.!RESET
- net +5V: now also M1.!SLP, M1.VDD(FLT), M2.!SLP, M2.VDD(FLT); no longer M1.!SLEEP, M1.VDD, M2.!SLEEP, M2.VDD
- net DEC-1A: now also M1.1A(A1); no longer M1.1A
- net DEC-1B: now also M1.1B(A2); no longer M1.1B
- net DEC-2A: now also M1.2A(B1); no longer M1.2A
- net DEC-2B: now also M1.2B(B2); no longer M1.2B
- net GND: now also PWM.SLEEVE, R22.1
- net IO0: now also R21.1, ST4.1
- net IO2: now also R21.2
- net MS1-1: now also SJ1.1; no longer M1.MS1
- net MS1-2: now also SJ2.1; no longer M2.MS1
- net MS2-1: now also M1.MS2(M1); no longer M1.MS2
- net MS2-2: now also M2.MS2(M1); no longer M2.MS2
- net MS3-1: now also M1.MS3(M2), SJ1.3; no longer M1.MS3
- net MS3-2: now also M2.MS3(M2), SJ2.3; no longer M2.MS3
- net RA-1A: now also M2.1A(A1); no longer M2.1A
- net RA-1B: now also M2.1B(A2); no longer M2.1B
- net RA-2A: now also M2.2A(B1); no longer M2.2A
- net RA-2B: now also M2.2B(B2); no longer M2.2B
- net V+: now also PWM.LEFT
Other:
- moved on the sheet: C10, C11, C12, D1, IC3, J1, PWR, R14
