File: AstroEQ-Hardware/PTH/AstroEQ PTH V4.7.sch (EAGLE design)
At the start: 52 parts, among them IC1 ATMEGA162-16PU-SKT, IC2 PIC18F14K50-I/P-SKT, IC3 78L05, M1 Motor Driver, M2 Motor Driver, Q1 NTR4501NT1G, X1 16MHz, X2 12MHz

Commit message: Update Hardware Designs
Minor corrections to part attributes and some components in the V4.7
design moved slightly to avoid collisions as found during the prototype
build.
Parts:
- added ICL1: ATMEGA162-16PU, ic-package:IC
- added ICL2: PIC18F14K50-I/P, ic-package:IC
- D2: value PMEG2010EA -> RB511VM-30FHTE-17; MF NEXPERIA -> ROHM; MPN PMEG2010EA -> RB511VM-30FHTE-17; OC_FARNELL 8737908 -> 2581544
- GPIO, J2, J3: value (none) -> DNI
- IC1: value ATMEGA162-16PU-SKT -> DIP40-SOCKET; MF ATMEL -> MULTICOMP; MPN ATMEGA162-16PU -> 2227MC-40-06-05-F1; OC_FARNELL 9171169 -> 1103855
- IC2: value PIC18F14K50-I/P-SKT -> DIP20-SOCKET; MF MICROCHIP -> MULTICOMP; MPN (none) -> 2227-20-03-07; OC_FARNELL (none) -> 4285608
- LOGO1: value ASTROEQ5MM -> DNI
- PROG: MF AMP - TE CONNECTIVITY -> HARWIN; MPN 826632-3 -> M20-9980346; OC_FARNELL 3418492 -> 1022231
- SJ1, SJ2: value (none) -> 3pin HDR; MF MULTICOMP -> HARWIN; MPN 2211S-03G -> M20-9990345.; OC_FARNELL 1593412 -> 1022248
Changed lines of the file:
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@@
 </part>
 <part name="GND5" library="supply1" deviceset="GND" device=""/>
-<part name="IC1" library="atmel" deviceset="ATMEGA162" device="-16PU-SKT" value="ATMEGA162-16PU-SKT">
-<attribute name="MF" value="ATMEL"/>
-<attribute name="MPN" value="ATMEGA162-16PU"/>
-<attribute name="OC_FARNELL" value="9171169"/>
-</part>
-<part name="IC2" library="microchip" deviceset="PIC18F14K50-I/P" device="-SKT" value="PIC18F14K50-I/P-SKT">
-<attribute name="MF" value="MICROCHIP"/>
+<part name="IC1" library="atmel" deviceset="ATMEGA162" device="-16PU-SKT" value="DIP40-SOCKET">
+<attribute name="MF" value="MULTICOMP"/>
+<attribute name="MPN" value="2227MC-40-06-05-F1"/>
+<attribute name="OC_FARNELL" value="1103855"/>
+</part>
+<part name="IC2" library="microchip" deviceset="PIC18F14K50-I/P" device="-SKT" value="DIP20-SOCKET">
+<attribute name="MF" value="MULTICOMP"/>
+<attribute name="MPN" value="2227-20-03-07"/>
+<attribute name="OC_FARNELL" value="4285608"/>
 </part>
 <part name="GND18" library="supply1" deviceset="GND" device=""/>
-<part name="D2" library="SparkFun" deviceset="DIODE" device="SOD" value="PMEG2010EA">
-<attribute name="MF" value="NEXPERIA"/>
-<attribute name="MPN" value="PMEG2010EA"/>
-<attribute name="OC_FARNELL" value="8737908"/>
+<part name="D2" library="SparkFun" deviceset="DIODE" device="SOD" value="RB511VM-30FHTE-17">
+<attribute name="MF" value="ROHM"/>
+<attribute name="MPN" value="RB511VM-30FHTE-17"/>
+<attribute name="OC_FARNELL" value="2581544"/>
 </part>
 <part name="GND19" library="supply1" deviceset="GND" device=""/>
@@
 <part name="GND16" library="supply1" deviceset="GND" device=""/>
 <part name="PROG" library="SparkFun" deviceset="AVR_SPI_PRG_6" device="PTH" value="AVR_PRG">
-<attribute name="MF" value="AMP - TE CONNECTIVITY"/>
-<attribute name="MPN" value="826632-3"/>
-<attribute name="OC_FARNELL" value="3418492"/>
+<attribute name="MF" value="HARWIN"/>
+<attribute name="MPN" value="M20-9980346"/>
+<attribute name="OC_FARNELL" value="1022231"/>
 </part>
 <part name="C11" library="rcl" deviceset="C-EU" device="C0603" value="100n">
@@
 <attribute name="OC_FARNELL" value="1536490"/>
 </part>
-<part name="GPIO" library="SparkFun" deviceset="M05" device="PTH">
+<part name="GPIO" library="SparkFun" deviceset="M05" device="PTH" value="DNI">
 <attribute name="MF" value=""/>
 <attribute name="MPN" value=""/>
@@
 </part>
 <part name="GND7" library="supply1" deviceset="GND" device=""/>
-<part name="LOGO1" library="CompanyLogos" deviceset="ASTROEQ" device="5MM">
+<part name="LOGO1" library="CompanyLogos" deviceset="ASTROEQ" device="5MM" value="DNI">
 <attribute name="MF" value=""/>
 <attribute name="MPN" value=""/>
@@
 <attribute name="OC_FARNELL" value="2447272"/>
 </part>
-<part name="SJ1" library="jumper" deviceset="JP2E" device="">
-<attribute name="MF" value="MULTICOMP"/>
-<attribute name="MPN" value="2211S-03G"/>
-<attribute name="OC_FARNELL" value="1593412"/>
-</part>
-<part name="SJ2" library="jumper" deviceset="JP2E" device="">
-<attribute name="MF" value="MULTICOMP"/>
-<attribute name="MPN" value="2211S-03G"/>
-<attribute name="OC_FARNELL" value="1593412"/>
-</part>
-<part name="J2" library="jumper" deviceset="JUMPER" device="">
+<part name="SJ1" library="jumper" deviceset="JP2E" device="" value="3pin HDR">
+<attribute name="MF" value="HARWIN"/>
+<attribute name="MPN" value="M20-9990345."/>
+<attribute name="OC_FARNELL" value="1022248"/>
+</part>
+<part name="SJ2" library="jumper" deviceset="JP2E" device="" value="3pin HDR">
+<attribute name="MF" value="HARWIN"/>
+<attribute name="MPN" value="M20-9990345."/>
+<attribute name="OC_FARNELL" value="1022248"/>
+</part>
+<part name="J2" library="jumper" deviceset="JUMPER" device="" value="DNI">
 <attribute name="MF" value="3M"/>
 <attribute name="MPN" value="969102-0000-DA"/>
 <attribute name="OC_FARNELL" value="2579814"/>
 </part>
-<part name="J3" library="jumper" deviceset="JUMPER" device="">
+<part name="J3" library="jumper" deviceset="JUMPER" device="" value="DNI">
 <attribute name="MF" value="3M"/>
 <attribute name="MPN" value="969102-0000-DA"/>
@@
 <attribute name="MPN" value="CES-116-01-T-S"/>
 <attribute name="OC_FARNELL" value="1667522"/>
+</part>
+<part name="ICL2" library="ic-package" deviceset="IC" device="" value="PIC18F14K50-I/P">
+<attribute name="MF" value="MICROCHIP"/>
+<attribute name="MPN" value="PIC18F14K50-I/P"/>
+<attribute name="OC_FARNELL" value="1648501"/>
+</part>
+<part name="ICL1" library="ic-package" deviceset="IC" device="" value="ATMEGA162-16PU">
+<attribute name="MF" value="ATMEL"/>
+<attribute name="MPN" value="ATMEGA162-16PU"/>
+<attribute name="OC_FARNELL" value="9171169"/>
 </part>
 </parts>
@@
 <attribute name="MPN" x="386.08" y="243.84" size="1.4224" layer="96" display="off"/>
 </instance>
+<instance part="ICL2" gate="G$1" x="81.28" y="266.7">
+<attribute name="OC_FARNELL" x="81.28" y="266.7" size="1.778" layer="96" display="off"/>
+<attribute name="MF" x="81.28" y="266.7" size="1.778" layer="96" display="off"/>
+<attribute name="MPN" x="81.28" y="266.7" size="1.778" layer="96" display="off"/>
+</instance>
+<instance part="ICL1" gate="G$1" x="241.3" y="264.16">
+<attribute name="OC_FARNELL" x="241.3" y="264.16" size="1.778" layer="96" display="off"/>
+<attribute name="MF" x="241.3" y="264.16" size="1.778" layer="96" display="off"/>
+<attribute name="MPN" x="241.3" y="264.16" size="1.778" layer="96" display="off"/>
+</instance>
 </instances>
