File: AstroEQ-Hardware/PTH/AstroEQ PTH V4.7.sch (EAGLE design)
At the start: 54 parts, among them IC1 DIP40-SOCKET, IC2 DIP20-SOCKET, IC3 78L05, J2 DNI, J3 DNI, M1 Motor Driver, M2 Motor Driver, Q1 NTR4501NT1G, X1 16MHz, X2 12MHz

Commit message: Update AstroEQ PTH/SMD Schematics
1. Tidy up the schematics, add a frame, and improve labelling of nets
2. Add extra textual documentation to the PCB to label the various extra IO pins.
Parts:
- IC1: device atmel:ATMEGA162-16PU-SKT -> atmel:ATMEGA162-16PU
- IC2: MPN 2227-20-03-07 -> (none); OC_FARNELL 4285608 -> (none)
Connections:
- net MISO renamed IO3-MISO
- net MOSI renamed ESTOP-MOSI
- net PWM-OUT renamed PWM-OD
- net SCLK renamed STAT-SCLK
Other:
- moved on the sheet: 12V, C1, C10, C11, C12, C13, C14, C15, C2, C3, C4, C5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
