File: AstroEQ-Hardware/PTH/AstroEQ PTH V4.6.brd (EAGLE design)
At the start: 100 x 66 mm, 56 parts, among them IC1 ATMEGA162-16PU, IC2 PIC18F14K50-I/P, IC3 78L05, J1 POWER_JACKPTH, M1 Motor Driver, M2 Motor Driver, Q1 BS270, X1 16MHz, X2 12MHz

Commit message: Update AstroEQ PTH/SMD Schematics
1. Tidy up the schematics, add a frame, and improve labelling of nets
2. Add extra textual documentation to the PCB to label the various extra IO pins.
Connections:
- net MISO renamed IO3-MISO
- net MOSI renamed ESTOP-MOSI
- net SCLK renamed STAT-SCLK
Other:
- board text added: "(wire to JP3)"
- board text added: "(wire to JP4)"
- board text added: "+5V IO0 IO1 IO2 GND"
- board text added: "ESTOP"
- board text added: "IO1 (SNAP)"
- board text added: "IO3 (SPEED)"
Changed lines of the file:
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@@
 <setting verticaltext="up"/>
 </settings>
-<grid distance="0.05" unitdist="inch" unit="inch" style="dots" multiple="1" display="yes" altdistance="0.0125" altunitdist="inch" altunit="inch"/>
+<grid distance="0.05" unitdist="inch" unit="mm" style="dots" multiple="1" display="yes" altdistance="0.0125" altunitdist="inch" altunit="mm"/>
 <layers>
 <layer number="1" name="Top" color="4" fill="1" visible="yes" active="yes"/>
 <layer number="2" name="Route2" color="1" fill="3" visible="no" active="no"/>
 <layer number="3" name="Route3" color="4" fill="3" visible="no" active="no"/>
+<layer number="4" name="Route4" color="1" fill="4" visible="no" active="no"/>
+<layer number="5" name="Route5" color="4" fill="4" visible="no" active="no"/>
+<layer number="6" name="Route6" color="1" fill="8" visible="no" active="no"/>
+<layer number="7" name="Route7" color="4" fill="8" visible="no" active="no"/>
+<layer number="8" name="Route8" color="1" fill="2" visible="no" active="no"/>
+<layer number="9" name="Route9" color="4" fill="2" visible="no" active="no"/>
+<layer number="10" name="Route10" color="1" fill="7" visible="no" active="no"/>
+<layer number="11" name="Route11" color="4" fill="7" visible="no" active="no"/>
+<layer number="12" name="Route12" color="1" fill="5" visible="no" active="no"/>
+<layer number="13" name="Route13" color="4" fill="5" visible="no" active="no"/>
 <layer number="14" name="Route14" color="1" fill="6" visible="no" active="no"/>
 <layer number="15" name="Route15" color="4" fill="6" visible="no" active="no"/>
@@
 <layer number="112" name="tSilk" color="7" fill="1" visible="no" active="yes"/>
 <layer number="113" name="ReferenceLS" color="7" fill="1" visible="no" active="yes"/>
+<layer number="114" name="PadCentre" color="7" fill="1" visible="yes" active="yes"/>
 <layer number="116" name="Patch_BOT" color="9" fill="4" visible="no" active="yes"/>
 <layer number="118" name="Rect_Pads" color="7" fill="1" visible="no" active="yes"/>
@@
 <layer number="131" name="tAdjust" color="7" fill="1" visible="no" active="yes"/>
 <layer number="132" name="bAdjust" color="7" fill="1" visible="no" active="yes"/>
+<layer number="133" name="Ports" color="7" fill="1" visible="no" active="yes"/>
+<layer number="134" name="Port2" color="7" fill="1" visible="no" active="yes"/>
+<layer number="135" name="Port3" color="7" fill="1" visible="no" active="yes"/>
 <layer number="144" name="Drill_legend" color="7" fill="1" visible="no" active="yes"/>
 <layer number="150" name="Top_Copper" color="7" fill="1" visible="no" active="yes"/>
@@
 <wire x1="89.535" y1="62.865" x2="85.09" y2="62.865" width="0.4064" layer="27" curve="-245.470453"/>
 <wire x1="85.09" y1="62.865" x2="89.535" y2="62.865" width="0.4064" layer="27"/>
+<wire x1="68.2625" y1="5.715" x2="65.7225" y2="5.715" width="0.4064" layer="27"/>
+<wire x1="68.2625" y1="3.175" x2="65.7225" y2="3.175" width="0.4064" layer="27"/>
+<wire x1="65.7225" y1="3.175" x2="65.7225" y2="5.715" width="0.4064" layer="27"/>
+<wire x1="68.2625" y1="5.715" x2="68.2625" y2="3.175" width="0.4064" layer="27"/>
+<wire x1="70.8025" y1="8.255" x2="68.2625" y2="8.255" width="0.4064" layer="27"/>
+<wire x1="70.8025" y1="5.715" x2="68.2625" y2="5.715" width="0.4064" layer="27"/>
+<wire x1="68.2625" y1="5.715" x2="68.2625" y2="8.255" width="0.4064" layer="27"/>
+<wire x1="70.8025" y1="8.255" x2="70.8025" y2="5.715" width="0.4064" layer="27"/>
+<text x="70.1675" y="1.905" size="1.2" layer="25" font="vector" ratio="15" align="center">IO3
+(SPEED)</text>
+<text x="65.7225" y="8.89" size="1.2" layer="25" font="vector" ratio="15" align="center">ESTOP</text>
+<text x="87.63" y="53.0225" size="0.7" layer="25" font="vector" ratio="15" align="center">(wire to
+ JP3)</text>
+<text x="47.3075" y="24.4475" size="0.7" layer="25" font="vector" ratio="15" rot="R90" align="center">(wire to JP4)</text>
+<text x="26.3525" y="13.97" size="1.2" layer="25" font="vector" ratio="15" rot="R180" align="center">+5V
+IO0
+IO1
+IO2
+GND</text>
+<wire x1="28.2575" y1="19.05" x2="24.4475" y2="19.05" width="0.4064" layer="27"/>
+<wire x1="28.2575" y1="8.89" x2="24.4475" y2="8.89" width="0.4064" layer="27"/>
+<wire x1="24.4475" y1="8.89" x2="24.4475" y2="19.05" width="0.4064" layer="27"/>
+<wire x1="28.2575" y1="19.05" x2="28.2575" y2="8.89" width="0.4064" layer="27"/>
+<text x="33.9725" y="28.575" size="1.2" layer="25" font="vector" ratio="15" rot="R90" align="center">IO1 (SNAP)</text>
+<wire x1="32.7025" y1="29.21" x2="31.4325" y2="29.21" width="0.4064" layer="27"/>
 </plain>
 <attributes>
@@
 </element>
 <element name="X2" library="SparkFun" package="HC49US" value="12MHz" x="18.7325" y="13.335" smashed="yes" rot="R180">
-<attribute name="NAME" x="25.2095" y="14.2875" size="1.016" layer="25" font="vector" ratio="15" rot="R270"/>
+<attribute name="NAME" x="10.795" y="12.827" size="1.016" layer="25" font="vector" ratio="15"/>
 <attribute name="OC_FARNELL" value="1842203" x="18.7325" y="13.335" size="1.778" layer="27" rot="R180" display="off"/>
 <attribute name="MF" value="TXC" x="18.7325" y="13.335" size="1.778" layer="27" rot="R180" display="off"/>
@@
 </element>
 <element name="M2" library="A4983Carrier" package="DIP16-W" value="Motor Driver" x="71.12" y="22.225" smashed="yes" rot="R270">
-<attribute name="NAME" x="63.8175" y="10.16" size="1.27" layer="25" font="vector" ratio="15"/>
+<attribute name="NAME" x="60.96" y="10.795" size="1.27" layer="25" font="vector" ratio="15"/>
 <attribute name="VALUE" x="79.375" y="30.7975" size="1.27" layer="27" font="vector" ratio="15" rot="R270"/>
 <attribute name="OC_FARNELL" value="1667522" x="71.12" y="22.225" size="1.778" layer="27" rot="R270" display="off"/>
@@
 <wire x1="58.42" y1="33.02" x2="58.7375" y2="33.02" width="0.6096" layer="16"/>
 </signal>
-<signal name="SCLK">
+<signal name="STAT-SCLK">
 <contactref element="R13" pad="1"/>
 <contactref element="IC1" pad="8"/>
@@
 <wire x1="31.13840625" y1="1.27" x2="37.465" y2="7.59659375" width="0.6096" layer="16"/>
 </signal>
-<signal name="MISO">
+<signal name="IO3-MISO">
 <contactref element="IC1" pad="7"/>
 <contactref element="PROG" pad="1"/>
@@
 <wire x1="65.0875" y1="4.445" x2="66.9925" y2="4.445" width="0.6096" layer="16"/>
 </signal>
-<signal name="MOSI">
+<signal name="ESTOP-MOSI">
 <contactref element="IC1" pad="6"/>
 <contactref element="PROG" pad="4"/>
@@
 </board>
 </drawing>
+<compatibility>
+<note version="6.3" minversion="6.2.2" severity="warning">
+Since Version 6.2.2 text objects can contain more than one line,
+which will not be processed correctly with this version.
+</note>
+</compatibility>
 </eagle>

Commit message: Update PTH V4.6 design missing USB connector shell connections
The USB connector shell pins were not being joined to the GND planes.
Connections:
- net GND: now also USB->.GND1, USB->.GND4
Changed lines of the file:
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@@
 <layer number="46" name="Milling" color="3" fill="1" visible="no" active="yes"/>
 <layer number="47" name="Measures" color="7" fill="1" visible="no" active="yes"/>
-<layer number="48" name="Document" color="7" fill="1" visible="no" active="yes"/>
-<layer number="49" name="Reference" color="7" fill="1" visible="no" active="yes"/>
+<layer number="48" name="Document" color="7" fill="1" visible="yes" active="yes"/>
+<layer number="49" name="Reference" color="7" fill="1" visible="yes" active="yes"/>
 <layer number="50" name="dxf" color="7" fill="1" visible="no" active="no"/>
 <layer number="51" name="tDocu" color="7" fill="1" visible="no" active="yes"/>
@@
 <via x="86.0425" y="55.88" extent="1-16" drill="0.6" shape="octagon"/>
 <via x="93.345" y="30.48" extent="1-16" drill="0.6" shape="octagon"/>
+<contactref element="USB-&gt;" pad="GND1"/>
+<contactref element="USB-&gt;" pad="GND4"/>
 </signal>
 <signal name="V+">
