File: AstroEQ-Hardware/PTH/AstroEQ PTH V4.8.sch (EAGLE design)
At the start: 55 parts, among them IC1 DIP40-SOCKET, IC2 DIP20-SOCKET, IC3 78L05, J2 DNI, J3 DNI, M1 Motor Driver, M2 Motor Driver, Q1 NTR4501NT1G, X1 16MHz, X2 12MHz

Commit message: Add target speed switch to EQ5 PCB
Other:
- note added: "IO3 selects between tracking speed on basic hand controller. Short = Solar Open = Sidereal 3.9kR = Lunar"
Changed lines of the file:
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@@
 <description>AstroEQ</description>
 <plain>
+<text x="20.32" y="91.44" size="1.4224" layer="97">IO3 selects between tracking
+speed on basic hand controller.
+Short = Solar
+Open = Sidereal
+3.9kR = Lunar</text>
 </plain>
 <instances>
@@
 <wire x1="73.66" y1="99.06" x2="68.58" y2="99.06" width="0.1524" layer="91"/>
 <junction x="68.58" y="99.06"/>
-</segment>
-</net>
+<wire x1="68.58" y1="106.68" x2="50.8" y2="106.68" width="0.1524" layer="91"/>
+<label x="50.8" y="106.68" size="1.4224" layer="95" font="vector" ratio="10" rot="R180" xref="yes"/>
+<junction x="68.58" y="106.68"/>
+</segment>
+</net>
