File: AstroEQ-Hardware/PTH/AstroEQ PTH V4.8.brd (EAGLE design)
At the start: 100 x 66 mm, 54 parts, among them IC1 ATMEGA162-16PU, IC2 PIC18F14K50-I/P, IC3 78L05, J1 POWER_JACKPTH, M1 Motor Driver, M2 Motor Driver, Q1 BS270, X1 16MHz, X2 12MHz

Commit message: Correct IO4 Pin on AstroEQ PCBs
Cannot use the Tx pin for this because the USB IC self-powers off this in standalone mode which prevents target speed selection.
Parts:
- R23: device rcl:0204/7 -> rcl:0207/10
- moved R23 1.27 mm to (48.3, 26.7)
Connections:
- new net IO4: IC1.21, R23.2
- net RX: no longer R23.2
Routing:
- net IO4: track 0.00 -> 37.0 mm, vias 0 -> 2
- net +5V: track 260.3 -> 263.8 mm
- net RX: track 37.4 -> 34.6 mm
- net RESET: track 88.2 -> 90.0 mm
- net MS2-2: track 52.4 -> 50.7 mm
- net MS3-2: track 57.4 -> 56.2 mm
- net TX: track 35.0 -> 35.9 mm
- net IO0: track 111.7 -> 112.5 mm
- net STEP-1: track 46.0 -> 46.8 mm
- net !RST-2: track 51.0 -> 50.2 mm
