File: AstroEQ-Hardware/DIY/AstroEQ DIY Etch.sch (EAGLE design)
At the start: 45 parts, among them IC1 ATMEGA162-16PU, IC2 PIC18F14K50-I/P, IC3 78L05, J1 POWER_JACKPTH, M1 Motor Driver, M2 Motor Driver, X1 16MHz, X2 12MHz

Commit message: Update AstroEQ DIY Design
The DIY version of the design (intended for home-etching on single-sided
PCB) was still V4.4. I have updated it to the V4.6 hardware.
Parts:
- added J2, J3: (no value), jumper:JUMPER
- added JP3, JP4: M01PTH, SparkFun:M01PTH
- added PWM: JACK, SparkFun:AUDIO-JACKPTH
- added Q1: BS270, SparkFun:MOSFET-NCHANNELPTH
- added R1: 10k, rcl:R-EU_0204/7
- added R21: 1k, rcl:R-EU_0204/7
- added R22: 120, rcl:R-EU_0204/7
- added SJ1: (no value), jumper:JP2E
- added SJ2: (no value), jumper:JP2EL
- D1: value C3D06065A -> MBR1060; MF CREE -> MULTICOMP; MPN C3D06065A -> MBR1060; OC_FARNELL 1864928 -> 1625119
- GPIO: MF (none) -> CYNERGY3; MPN (none) -> SSF211X050; OC_FARNELL (none) -> 4249100
- HAMMOND-1593N: value HAMMOND-1593N -> HAMMOND-1593N-4HOLE; device holes:HAMMOND-1593N -> holes:HAMMOND-1593N-4HOLE
- JP1, JP2: OC_FARNELL (none) -> unknown
- LOGO1: value ASTROEQ3MM -> ASTROEQ5MM; device CompanyLogos:ASTROEQ3MM -> CompanyLogos:ASTROEQ5MM; OC_FARNELL (none) -> unknown
- ST4: MF (none) -> MOLEX; MPN (none) -> 95501-2661; OC_FARNELL (none) -> 1536490
Connections:
- removed net DEC+B: JP2.2, ST4.5
- removed net DEC-B: JP2.3, ST4.4
- removed net RA+B: JP2.1, ST4.6
- removed net RA-B: JP2.4, ST4.3
- new net DEC+/SI: IC1.PA6/AD6/PCINT6, JP1.2
- new net DEC-/CK: IC1.PA5/AD5/PCINT5, JP1.3
- new net MS13-1: M1.MS1(M0), SJ1.2
- new net MS13-2: M2.MS1(M0), SJ2.2
- new net PWM: IC1.PB1/T1/OC2, JP3.1
- new net PWM-ILIM: Q1.S, R22.2
- new net PWM-OUT: PWM.RIGHT, Q1.D
- new net PWM-Q1: JP4.1, Q1.G
- new net RA+/SO: IC1.PA7/AD7/PCINT7, JP1.1
- new net RA-/!SS: IC1.PA4/AD4/PCINT4, JP1.4
- net !RST-1: now also M1.!RST; no longer M1.!RESET
- net !RST-2: now also M2.!RST; no longer M2.!RESET
- net +5V: now also M1.!SLP, M1.VDD(FLT), M2.!SLP, M2.VDD(FLT); no longer M1.!SLEEP, M1.VDD, M2.!SLEEP, M2.VDD
- net DEC+: now also JP2.2, ST4.5; no longer IC1.PA6/AD6/PCINT6, JP1.2
- net DEC-: now also JP2.3, ST4.4; no longer IC1.PA5/AD5/PCINT5, JP1.3
- net DEC-1A: now also M1.1A(A1); no longer M1.1A
- net DEC-1B: now also M1.1B(A2); no longer M1.1B
- net DEC-2A: now also M1.2A(B1); no longer M1.2A
- net DEC-2B: now also M1.2B(B2); no longer M1.2B
- net DTR: now also R1.1
- net GND: now also PWM.SLEEVE, R1.2, R22.1
- net IO0: now also R21.1, ST4.1
- net IO2: now also R21.2
- net MS1-1: now also SJ1.1; no longer M1.MS1
- net MS1-2: now also SJ2.1; no longer M2.MS1
- net MS2-1: now also M1.MS2(M1); no longer M1.MS2
- net MS2-2: now also M2.MS2(M1); no longer M2.MS2
- net MS3-1: now also M1.MS3(M2), SJ1.3; no longer M1.MS3
- net MS3-2: now also M2.MS3(M2), SJ2.3; no longer M2.MS3
- net RA+: now also JP2.1, ST4.6; no longer IC1.PA7/AD7/PCINT7, JP1.1
- net RA-: now also JP2.4, ST4.3; no longer IC1.PA4/AD4/PCINT4, JP1.4
- net RA-1A: now also M2.1A(A1); no longer M2.1A
- net RA-1B: now also M2.1B(A2); no longer M2.1B
- net RA-2A: now also M2.2A(B1); no longer M2.2A
- net RA-2B: now also M2.2B(B2); no longer M2.2B
- net V+: now also PWM.LEFT
Other:
- moved on the sheet: C10, C11, C12, D1, IC3, J1, PWR, R14
