File: AstroEQ-Hardware/DIY/AstroEQ DIY Etch.sch (EAGLE design)
At the start: 57 parts, among them IC1 ATMEGA162-16PU, IC2 PIC18F14K50-I/P, IC3 78L05, J1 POWER_JACKPTH, M1 Motor Driver, M2 Motor Driver, Q1 BS270, X1 16MHz, X2 12MHz

Commit message: Correct IO4 Pin on AstroEQ PCBs
Cannot use the Tx pin for this because the USB IC self-powers off this in standalone mode which prevents target speed selection.
Parts:
- R23: device rcl:R-EU_0204/7 -> rcl:R-EU_0207/10
Connections:
- new net IO4: IC1.PC0/A8/PCINT8, R23.2
- net RX: no longer R23.2
