File: AstroEQ-Hardware/DIY/AstroEQ DIY Etch.brd (EAGLE design)
At the start: 100 x 66 mm, 56 parts, among them IC1 ATMEGA162-16PU, IC2 PIC18F14K50-I/P, IC3 78L05, J1 POWER_JACKPTH, M1 Motor Driver, M2 Motor Driver, Q1 BS270, X1 16MHz, X2 12MHz

Commit message: Update DIY Etch Schematic Formatting (no actual design changes)
Tidy up the schematic and add frame to match the PTH V4.6 tidy up
Connections:
- net MISO renamed IO3-MISO
- net MOSI renamed ESTOP-MOSI
- net SCLK renamed STAT-SCLK
Changed lines of the file:
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@@
 <setting verticaltext="up"/>
 </settings>
-<grid distance="0.05" unitdist="inch" unit="inch" style="dots" multiple="1" display="yes" altdistance="0.0125" altunitdist="inch" altunit="inch"/>
+<grid distance="0.05" unitdist="inch" unit="mm" style="dots" multiple="1" display="yes" altdistance="0.0125" altunitdist="inch" altunit="mm"/>
 <layers>
 <layer number="1" name="Top" color="4" fill="1" visible="yes" active="yes"/>
 <layer number="2" name="Route2" color="1" fill="3" visible="no" active="no"/>
 <layer number="3" name="Route3" color="4" fill="3" visible="no" active="no"/>
+<layer number="4" name="Route4" color="1" fill="4" visible="no" active="yes"/>
+<layer number="5" name="Route5" color="4" fill="4" visible="no" active="yes"/>
+<layer number="6" name="Route6" color="1" fill="8" visible="no" active="yes"/>
+<layer number="7" name="Route7" color="4" fill="8" visible="no" active="yes"/>
+<layer number="8" name="Route8" color="1" fill="2" visible="no" active="yes"/>
+<layer number="9" name="Route9" color="4" fill="2" visible="no" active="yes"/>
+<layer number="10" name="Route10" color="1" fill="7" visible="no" active="yes"/>
+<layer number="11" name="Route11" color="4" fill="7" visible="no" active="yes"/>
+<layer number="12" name="Route12" color="1" fill="5" visible="no" active="yes"/>
+<layer number="13" name="Route13" color="4" fill="5" visible="no" active="yes"/>
 <layer number="14" name="Route14" color="1" fill="6" visible="no" active="no"/>
 <layer number="15" name="Route15" color="4" fill="6" visible="no" active="no"/>
@@
 <wire x1="58.42" y1="33.02" x2="58.7375" y2="33.02" width="0.6096" layer="16"/>
 </signal>
-<signal name="SCLK">
+<signal name="STAT-SCLK">
 <contactref element="R13" pad="1"/>
 <contactref element="IC1" pad="8"/>
@@
 <wire x1="31.13840625" y1="1.27" x2="37.465" y2="7.59659375" width="0.6096" layer="16"/>
 </signal>
-<signal name="MISO">
+<signal name="IO3-MISO">
 <contactref element="IC1" pad="7"/>
 <contactref element="PROG" pad="1"/>
@@
 <wire x1="65.0875" y1="4.445" x2="66.9925" y2="4.445" width="0.6096" layer="16"/>
 </signal>
-<signal name="MOSI">
+<signal name="ESTOP-MOSI">
 <contactref element="IC1" pad="6"/>
 <contactref element="PROG" pad="4"/>

Commit message: Add extra target speed resistor to AstroEQ DIY
Bump version to hardware V4.8
Parts:
- added R23: 1k, rcl:0204/7
- SJ1: device jumper:JP2 -> jumper:JP2L
- moved JP3 12.7 mm to (47.9, 6.35)
Connections:
- net IO3-MISO: now also R23.1
- net RX: now also R23.2
Routing:
- net PWM: track 21.8 -> 2.86 mm
- net IO0: track 97.4 -> 113.8 mm, vias 4 -> 2
- net IO3-MISO: track 49.3 -> 36.0 mm, vias 0 -> 2
- net MS3-1: track 55.6 -> 64.0 mm
- net !EN-1: track 69.7 -> 65.9 mm
- net RX: track 34.3 -> 37.4 mm
- net STAT-SCLK: track 87.4 -> 85.6 mm
- net MS2-1: track 51.2 -> 49.9 mm
- net ESTOP-MOSI: track 38.5 -> 37.4 mm
- net !RST-2: track 51.8 -> 51.0 mm
- net RESET: track 88.8 -> 88.2 mm
- net MS3-2: track 58.0 -> 57.4 mm
- net MS2-2: track 51.9 -> 52.4 mm
- net !RST-1: track 67.8 -> 68.4 mm
Other:
- board text added: "(C) 2012-26"
- board text added: "V4.8-DIY"
- board text added: "V4.8-PTH"
- board text removed: "(C) 2012-16"
- board text removed: "V4.6-DIY"
- board text removed: "V4.6-PTH"

Commit message: Update DIY Silk and Routing
Improve silk and slightly tweak the routing.
Routing:
- net IO0: track 113.8 -> 111.7 mm
- net +5V: track 259.2 -> 260.3 mm
Other:
- board text added: "(wire to JP3)"
- board text added: "(wire to JP4)"
- board text added: "+5V IO0 IO1 IO2 GND"
- board text added: "ESTOP"
- board text added: "IO1 (SNAP)"
- board text added: "IO3 (SPEED)"

Commit message: Correct IO4 Pin on AstroEQ PCBs
Cannot use the Tx pin for this because the USB IC self-powers off this in standalone mode which prevents target speed selection.
Parts:
- R23: device rcl:0204/7 -> rcl:0207/10
- moved R23 1.27 mm to (48.3, 26.7)
Connections:
- new net IO4: IC1.21, R23.2
- net RX: no longer R23.2
Routing:
- net IO4: track 0.00 -> 37.0 mm, vias 0 -> 2
- net RX: track 37.4 -> 34.6 mm
- net RESET: track 88.2 -> 90.0 mm
- net MS2-2: track 52.4 -> 50.7 mm
- net MS3-2: track 57.4 -> 56.2 mm
- net TX: track 35.0 -> 35.9 mm
- net STEP-1: track 46.0 -> 46.8 mm
- net !RST-2: track 51.0 -> 50.2 mm
- net IO0: track 111.7 -> 111.2 mm
