File: AstroEQ-Hardware/EQ5/AstroEQ SMD V4.8 (EQ5).brd (EAGLE design)
At the start: 85 x 49 mm, 56 parts, among them IC1 ATMEGA162-16AU, IC2 PIC18F14K50-I/SS, IC3 78L05, J1 POWER_JACKPANEL, J2 DNI, J3 DNI, M1 Motor Driver, M2 Motor Driver, Q1 NTR4501NT1G, Q2 NTR4501NT1G, X1 16MHz, X2 12MHz

Commit message: Add target speed switch to EQ5 PCB
Parts:
- removed HC-SPEED: JS102011SAQN, SparkFun:SWITCH-SPDT-SMD
- added HCSPEED: SLW-1277545-2A-RA-D, switch:SLW-127
- added R2: 3.9k, rcl:R0603
- added R23: 1k, rcl:R0603
- moved C5 0.32 mm to (7.30, 23.5)
Connections:
- new net N$1: HCSPEED.1, R2.1
- net GND: now also HCSPEED.5, HCSPEED.S1, HCSPEED.S2, R2.2; no longer HC-SPEED.2, HC-SPEED.3
- net IO3-MISO: now also HCSPEED.3, R23.2; no longer HC-SPEED.1
- net RX: now also R23.1
Routing:
- net VPIC: track 47.8 -> 43.6 mm
- net IO3-MISO: track 63.9 -> 68.0 mm, vias 1 -> 2
- net N$1: track 0.00 -> 3.39 mm
- net RX: track 16.8 -> 18.3 mm
- net GND: vias 166 -> 168

Commit message: Correct IO4 Pin on AstroEQ PCBs
Cannot use the Tx pin for this because the USB IC self-powers off this in standalone mode which prevents target speed selection.
Parts:
- moved R23 21.3 mm to (15.2, 14.6), flipped to the bottom, turned to 90 degrees
Connections:
- new net IO4: IC1.18, R23.1
- net AVROSC1: now also X1.1; no longer X1.P$1
- net AVROSC2: now also X1.2; no longer X1.P$2
- net RX: no longer R23.1
- net USBOSC1: now also X2.2; no longer X2.P$2
- net USBOSC2: now also X2.1; no longer X2.P$1
Routing:
- net IO4: track 0.00 -> 31.5 mm
- net RA-/!SS: track 31.5 -> 33.7 mm
- net RX: track 18.3 -> 16.8 mm
- net DEC-/CK: track 34.4 -> 35.2 mm
- net IO3-MISO: track 68.0 -> 67.5 mm, vias 2 -> 1
- net GND: vias 168 -> 172
