File: AstroEQ-Hardware/EQ5/AstroEQ SMD V4.8 (EQ5).sch (EAGLE design)
At the start: 56 parts, among them IC1 ATMEGA162-16AU, IC2 PIC18F14K50-I/SS, IC3 78L05, J1 POWER_JACKPANEL, J2 DNI, J3 DNI, M1 Motor Driver, M2 Motor Driver, Q1 NTR4501NT1G, Q2 NTR4501NT1G, X1 16MHz, X2 12MHz

Commit message: Add target speed switch to EQ5 PCB
Parts:
- removed HC-SPEED: JS102011SAQN, SparkFun:SWITCH-SPSTSMD2
- added HCSPEED: SLW-1277545-2A-RA-D, switch:SLW-1277545-2A-RA-D
- added R2: 3.9k, rcl:R-EU_R0603
- added R23: 1k, rcl:R-EU_R0603
Connections:
- new net N$1: HCSPEED.S, R2.1
- net GND: now also HCSPEED.O, HCSPEED.SH, R2.2; no longer HC-SPEED.P, HC-SPEED.S
- net IO3-MISO: now also HCSPEED.P, R23.2; no longer HC-SPEED.O
- net RX: now also R23.1
Other:
- note added: "Selects between tracking speed on basic hand controller. Short = Solar Open = Sidereal 3.9kR = Lunar"
- note removed: "Selects between tracking speed ranges on basic hand controller. Open = Sidereal/2x Sid/GoTo Speed Closed = Sidereal/Solar/Lunar"
Changed lines of the file:
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@@
 <attribute name="OC_FARNELL" value="1229685"/>
-</part>
-<part name="HC-SPEED" library="SparkFun" deviceset="SWITCH-SPST" device="SMD2" value="JS102011SAQN">
-<attribute name="MANUFACTURER" value="MF"/>
-<attribute name="OC_FARNELL" value="2320017"/>
 </part>
 <part name="GND8" library="supply1" deviceset="GND" device=""/>
@@
 </part>
 <part name="GND12" library="supply1" deviceset="GND" device=""/>
+<part name="R2" library="rcl" deviceset="R-EU_" device="R0603" value="3.9k">
+<attribute name="MF" value="MULTICOMP"/>
+<attribute name="MPN" value="MCWR06X1001FTL"/>
+<attribute name="OC_FARNELL" value="2447272"/>
+</part>
+<part name="R23" library="rcl" deviceset="R-EU_" device="R0603" value="1k">
+<attribute name="MF" value="MULTICOMP"/>
+<attribute name="MPN" value="MCWR06X1001FTL"/>
+<attribute name="OC_FARNELL" value="2447272"/>
+</part>
+<part name="HCSPEED" library="switch" deviceset="SLW-127" device="7545-2A-RA-D"/>
 </parts>
 <sheets>
@@
 pins connected to make routing easier.
 Use 6P4C cable. or ignore outer two pins</text>
-<text x="119.38" y="147.32" size="1.4224" layer="97">Selects between tracking speed ranges
+<text x="119.38" y="147.32" size="1.4224" layer="97">Selects between tracking speed
 on basic hand controller.
-Open = Sidereal/2x Sid/GoTo Speed
-Closed = Sidereal/Solar/Lunar</text>
+Short = Solar
+Open = Sidereal
+3.9kR = Lunar</text>
 </plain>
 <instances>
@@
 </instance>
 <instance part="GND7" gate="1" x="195.58" y="127"/>
-<instance part="HC-SPEED" gate="1" x="139.7" y="137.16" rot="R180">
-<attribute name="OC_FARNELL" x="139.7" y="137.16" size="1.4224" layer="96" font="vector" ratio="10" rot="R180" align="center" display="off"/>
-<attribute name="MANUFACTURER" x="139.7" y="137.16" size="1.4224" layer="96" font="vector" ratio="10" rot="R180" align="center" display="off"/>
-</instance>
-<instance part="GND8" gate="1" x="144.78" y="127"/>
+<instance part="GND8" gate="1" x="160.02" y="129.54"/>
 <instance part="EXT-IO" gate="G$1" x="22.86" y="142.24" rot="MR180">
 <attribute name="OC_FARNELL" x="22.86" y="142.24" size="1.778" layer="96" display="off"/>
@@
 </instance>
 <instance part="GND12" gate="1" x="73.66" y="25.4"/>
+<instance part="R2" gate="G$1" x="149.86" y="134.62" smashed="yes">
+<attribute name="NAME" x="150.876" y="138.0744" size="1.778" layer="95" rot="R180"/>
+<attribute name="VALUE" x="152.4" y="133.477" size="1.778" layer="96" rot="R180"/>
+<attribute name="OC_FARNELL" value="9342400" x="149.86" y="134.62" size="1.778" layer="96" rot="R90" display="off"/>
+<attribute name="MF" value="MULTICOMP" x="149.86" y="134.62" size="1.778" layer="96" rot="R90" display="off"/>
+<attribute name="MPN" value="MF12 1K" x="149.86" y="134.62" size="1.778" layer="96" rot="R90" display="off"/>
+</instance>
+<instance part="R23" gate="G$1" x="114.3" y="137.16" smashed="yes">
+<attribute name="NAME" x="115.316" y="140.6144" size="1.778" layer="95" rot="R180"/>
+<attribute name="VALUE" x="116.84" y="136.017" size="1.778" layer="96" rot="R180"/>
+<attribute name="OC_FARNELL" value="9342400" x="114.3" y="137.16" size="1.778" layer="96" rot="R90" display="off"/>
+<attribute name="MF" value="MULTICOMP" x="114.3" y="137.16" size="1.778" layer="96" rot="R90" display="off"/>
+<attribute name="MPN" value="MF12 1K" x="114.3" y="137.16" size="1.778" layer="96" rot="R90" display="off"/>
+</instance>
+<instance part="HCSPEED" gate="G$1" x="129.54" y="137.16" rot="R270"/>
 </instances>
 <busses>
@@
 </segment>
 <segment>
-<pinref part="HC-SPEED" gate="1" pin="S"/>
-<wire x1="134.62" y1="139.7" x2="132.08" y2="139.7" width="0.1524" layer="91"/>
-<wire x1="132.08" y1="139.7" x2="132.08" y2="144.78" width="0.1524" layer="91"/>
-<wire x1="132.08" y1="144.78" x2="144.78" y2="144.78" width="0.1524" layer="91"/>
-<pinref part="HC-SPEED" gate="1" pin="P"/>
-<wire x1="144.78" y1="137.16" x2="144.78" y2="129.54" width="0.1524" layer="91"/>
-<wire x1="142.24" y1="137.16" x2="144.78" y2="137.16" width="0.1524" layer="91"/>
-<wire x1="144.78" y1="137.16" x2="144.78" y2="144.78" width="0.1524" layer="91"/>
+<wire x1="134.62" y1="139.7" x2="137.16" y2="139.7" width="0.1524" layer="91"/>
+<wire x1="137.16" y1="139.7" x2="160.02" y2="139.7" width="0.1524" layer="91"/>
+<wire x1="160.02" y1="132.08" x2="160.02" y2="134.62" width="0.1524" layer="91"/>
 <pinref part="GND8" gate="1" pin="GND"/>
-<junction x="144.78" y="137.16"/>
+<junction x="160.02" y="134.62"/>
+<wire x1="160.02" y1="134.62" x2="160.02" y2="139.7" width="0.1524" layer="91"/>
+<pinref part="R2" gate="G$1" pin="2"/>
+<wire x1="154.94" y1="134.62" x2="160.02" y2="134.62" width="0.1524" layer="91"/>
+<pinref part="HCSPEED" gate="G$1" pin="O"/>
+<pinref part="HCSPEED" gate="G$1" pin="SH"/>
+<wire x1="124.46" y1="139.7" x2="121.92" y2="139.7" width="0.1524" layer="91"/>
+<wire x1="121.92" y1="139.7" x2="121.92" y2="142.24" width="0.1524" layer="91"/>
+<wire x1="121.92" y1="142.24" x2="137.16" y2="142.24" width="0.1524" layer="91"/>
+<wire x1="137.16" y1="142.24" x2="137.16" y2="139.7" width="0.1524" layer="91"/>
+<junction x="137.16" y="139.7"/>
 </segment>
 <segment>
@@
 <segment>
 <pinref part="IC1" gate="G$1" pin="PD0/RXD0"/>
-<wire x1="142.24" y1="91.44" x2="55.88" y2="91.44" width="0.1524" layer="91"/>
 <label x="139.7" y="91.44" size="1.778" layer="95" rot="MR0"/>
 <label x="55.88" y="91.44" size="1.4224" layer="95" font="vector" ratio="10" rot="R180" xref="yes"/>
+<wire x1="142.24" y1="91.44" x2="55.88" y2="91.44" width="0.1524" layer="91"/>
 </segment>
 <segment>
@@
 <segment>
 <pinref part="IC1" gate="G$1" pin="PD1/TXD0"/>
-<wire x1="142.24" y1="88.9" x2="55.88" y2="88.9" width="0.1524" layer="91"/>
+<wire x1="142.24" y1="88.9" x2="106.68" y2="88.9" width="0.1524" layer="91"/>
 <label x="139.7" y="88.9" size="1.778" layer="95" rot="MR0"/>
 <label x="55.88" y="88.9" size="1.4224" layer="95" font="vector" ratio="10" rot="R180" xref="yes"/>
+<junction x="106.68" y="88.9"/>
+<wire x1="106.68" y1="88.9" x2="55.88" y2="88.9" width="0.1524" layer="91"/>
+<pinref part="R23" gate="G$1" pin="1"/>
+<wire x1="109.22" y1="137.16" x2="106.68" y2="137.16" width="0.1524" layer="91"/>
+<wire x1="106.68" y1="137.16" x2="106.68" y2="88.9" width="0.1524" layer="91"/>
 </segment>
 <segment>
@@
 <wire x1="76.2" y1="104.14" x2="121.92" y2="104.14" width="0.1524" layer="91"/>
 <label x="139.7" y="104.14" size="1.778" layer="95" rot="MR0"/>
-<pinref part="HC-SPEED" gate="1" pin="O"/>
 <wire x1="121.92" y1="104.14" x2="142.24" y2="104.14" width="0.1524" layer="91"/>
-<wire x1="121.92" y1="104.14" x2="121.92" y2="134.62" width="0.1524" layer="91"/>
-<wire x1="121.92" y1="134.62" x2="134.62" y2="134.62" width="0.1524" layer="91"/>
+<wire x1="121.92" y1="104.14" x2="121.92" y2="137.16" width="0.1524" layer="91"/>
 <junction x="121.92" y="104.14"/>
+<wire x1="124.46" y1="137.16" x2="121.92" y2="137.16" width="0.1524" layer="91"/>
+<pinref part="R23" gate="G$1" pin="2"/>
+<wire x1="119.38" y1="137.16" x2="121.92" y2="137.16" width="0.1524" layer="91"/>
+<junction x="121.92" y="137.16"/>
+<pinref part="HCSPEED" gate="G$1" pin="P"/>
 </segment>
 </net>
@@
 </segment>
 </net>
+<net name="N$1" class="0">
+<segment>
+<pinref part="R2" gate="G$1" pin="1"/>
+<wire x1="144.78" y1="134.62" x2="134.62" y2="134.62" width="0.1524" layer="91"/>
+<pinref part="HCSPEED" gate="G$1" pin="S"/>
+</segment>
+</net>

Commit message: Correct IO4 Pin on AstroEQ PCBs
Cannot use the Tx pin for this because the USB IC self-powers off this in standalone mode which prevents target speed selection.
Connections:
- new net IO4: IC1.PC0/A8/PCINT8, R23.1
- net RX: no longer R23.1
Other:
- moved on the sheet: R23
Changed lines of the file:
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@@
 <attribute name="MPN" value="MF12 1K" x="149.86" y="134.62" size="1.778" layer="96" rot="R90" display="off"/>
 </instance>
-<instance part="R23" gate="G$1" x="114.3" y="137.16" smashed="yes">
-<attribute name="NAME" x="115.316" y="140.6144" size="1.778" layer="95" rot="R180"/>
-<attribute name="VALUE" x="116.84" y="136.017" size="1.778" layer="96" rot="R180"/>
-<attribute name="OC_FARNELL" value="9342400" x="114.3" y="137.16" size="1.778" layer="96" rot="R90" display="off"/>
-<attribute name="MF" value="MULTICOMP" x="114.3" y="137.16" size="1.778" layer="96" rot="R90" display="off"/>
-<attribute name="MPN" value="MF12 1K" x="114.3" y="137.16" size="1.778" layer="96" rot="R90" display="off"/>
+<instance part="R23" gate="G$1" x="121.92" y="124.46" smashed="yes" rot="R180">
+<attribute name="NAME" x="120.904" y="121.0056" size="1.778" layer="95"/>
+<attribute name="VALUE" x="119.38" y="125.603" size="1.778" layer="96"/>
+<attribute name="OC_FARNELL" value="9342400" x="121.92" y="124.46" size="1.778" layer="96" rot="R270" display="off"/>
+<attribute name="MF" value="MULTICOMP" x="121.92" y="124.46" size="1.778" layer="96" rot="R270" display="off"/>
+<attribute name="MPN" value="MF12 1K" x="121.92" y="124.46" size="1.778" layer="96" rot="R270" display="off"/>
 </instance>
 <instance part="HCSPEED" gate="G$1" x="129.54" y="137.16" rot="R270"/>
@@
 <segment>
 <pinref part="IC1" gate="G$1" pin="PD1/TXD0"/>
-<wire x1="142.24" y1="88.9" x2="106.68" y2="88.9" width="0.1524" layer="91"/>
 <label x="139.7" y="88.9" size="1.778" layer="95" rot="MR0"/>
 <label x="55.88" y="88.9" size="1.4224" layer="95" font="vector" ratio="10" rot="R180" xref="yes"/>
-<junction x="106.68" y="88.9"/>
-<wire x1="106.68" y1="88.9" x2="55.88" y2="88.9" width="0.1524" layer="91"/>
-<pinref part="R23" gate="G$1" pin="1"/>
-<wire x1="109.22" y1="137.16" x2="106.68" y2="137.16" width="0.1524" layer="91"/>
-<wire x1="106.68" y1="137.16" x2="106.68" y2="88.9" width="0.1524" layer="91"/>
+<wire x1="142.24" y1="88.9" x2="55.88" y2="88.9" width="0.1524" layer="91"/>
 </segment>
 <segment>
@@
 <wire x1="78.74" y1="71.12" x2="76.2" y2="71.12" width="0.1524" layer="91"/>
 <wire x1="76.2" y1="71.12" x2="76.2" y2="104.14" width="0.1524" layer="91"/>
-<wire x1="76.2" y1="104.14" x2="121.92" y2="104.14" width="0.1524" layer="91"/>
+<wire x1="76.2" y1="104.14" x2="114.3" y2="104.14" width="0.1524" layer="91"/>
 <label x="139.7" y="104.14" size="1.778" layer="95" rot="MR0"/>
-<wire x1="121.92" y1="104.14" x2="142.24" y2="104.14" width="0.1524" layer="91"/>
-<wire x1="121.92" y1="104.14" x2="121.92" y2="137.16" width="0.1524" layer="91"/>
-<junction x="121.92" y="104.14"/>
-<wire x1="124.46" y1="137.16" x2="121.92" y2="137.16" width="0.1524" layer="91"/>
+<wire x1="114.3" y1="104.14" x2="142.24" y2="104.14" width="0.1524" layer="91"/>
+<wire x1="114.3" y1="104.14" x2="114.3" y2="124.46" width="0.1524" layer="91"/>
+<junction x="114.3" y="104.14"/>
+<wire x1="124.46" y1="137.16" x2="114.3" y2="137.16" width="0.1524" layer="91"/>
+<wire x1="114.3" y1="137.16" x2="114.3" y2="124.46" width="0.1524" layer="91"/>
 <pinref part="R23" gate="G$1" pin="2"/>
-<wire x1="119.38" y1="137.16" x2="121.92" y2="137.16" width="0.1524" layer="91"/>
-<junction x="121.92" y="137.16"/>
+<wire x1="116.84" y1="124.46" x2="114.3" y2="124.46" width="0.1524" layer="91"/>
+<junction x="114.3" y="124.46"/>
 <pinref part="HCSPEED" gate="G$1" pin="P"/>
 </segment>
@@
 <label x="99.06" y="152.4" size="1.778" layer="95"/>
 <pinref part="Q1" gate="G$1" pin="G"/>
-<wire x1="99.06" y1="152.4" x2="101.6" y2="152.4" width="0.1524" layer="91"/>
-<wire x1="101.6" y1="152.4" x2="101.6" y2="116.84" width="0.1524" layer="91"/>
+<wire x1="99.06" y1="152.4" x2="106.68" y2="152.4" width="0.1524" layer="91"/>
+<wire x1="106.68" y1="152.4" x2="106.68" y2="116.84" width="0.1524" layer="91"/>
 <pinref part="IC1" gate="G$1" pin="PB1/T1/OC2"/>
-<wire x1="101.6" y1="116.84" x2="142.24" y2="116.84" width="0.1524" layer="91"/>
+<wire x1="106.68" y1="116.84" x2="142.24" y2="116.84" width="0.1524" layer="91"/>
 <label x="139.7" y="116.84" size="1.778" layer="95" rot="MR0"/>
 </segment>
@@
 <junction x="226.06" y="15.24"/>
 <label x="231.14" y="15.24" size="1.4224" layer="95" xref="yes"/>
-</segment>
-</net>
-<net name="!NOT-ALLOWED!" class="0">
-<segment>
-<wire x1="210.82" y1="93.98" x2="215.9" y2="93.98" width="0.1524" layer="91"/>
-<wire x1="215.9" y1="93.98" x2="215.9" y2="71.12" width="0.1524" layer="91"/>
-<wire x1="215.9" y1="71.12" x2="210.82" y2="71.12" width="0.1524" layer="91"/>
-<label x="218.44" y="73.66" size="1.778" layer="95" rot="R90"/>
-<wire x1="210.82" y1="93.98" x2="210.82" y2="94.234" width="0.1524" layer="91"/>
-<wire x1="210.82" y1="94.234" x2="216.154" y2="94.234" width="0.1524" layer="91"/>
-<wire x1="216.154" y1="94.234" x2="216.154" y2="70.866" width="0.1524" layer="91"/>
-<wire x1="216.154" y1="70.866" x2="210.82" y2="70.866" width="0.1524" layer="91"/>
-<wire x1="210.82" y1="70.866" x2="210.82" y2="71.12" width="0.1524" layer="91"/>
 </segment>
 </net>
@@
 </segment>
 </net>
+<net name="IO4" class="0">
+<segment>
+<pinref part="R23" gate="G$1" pin="1"/>
+<wire x1="127" y1="124.46" x2="129.54" y2="124.46" width="0.1524" layer="91"/>
+<label x="129.54" y="124.46" size="1.4224" layer="95" font="vector" ratio="10" xref="yes"/>
+</segment>
+<segment>
+<wire x1="213.36" y1="91.44" x2="215.9" y2="91.44" width="0.1524" layer="91"/>
+<label x="215.9" y="91.44" size="1.4224" layer="95" font="vector" ratio="10" xref="yes"/>
+<pinref part="IC1" gate="G$1" pin="PC0/A8/PCINT8"/>
+</segment>
+</net>
